Commit message: Temp fix: fixed wheels

File: scout_description/urdf/scout_mini_wheel.xacro (robot description, xacro)
@@ -24,5 +24,5 @@
             </collision>
         </link>
-        <joint name="${wheel_prefix}_wheel" type="continuous">
+        <joint name="${wheel_prefix}_wheel" type="fixed">
             <parent link="${parent_link}"/>
             <child link="${wheel_prefix}_wheel_link"/>
